Commit message: create collision in robot_description

File: robot_description/urdf/base_link.xacro (robot description, xacro)
@@ -10,4 +10,20 @@
             <origin xyz="0 0 0" rpy="0 0 0"/>
         </visual>
+        <collision>
+            <geometry>
+                <mesh filename="package://robot_description/meshes/chassis.stl" scale="1 1 1" />
+            </geometry>
+            <surface>
+                <friction>
+                    <ode>
+                        <mu>0</mu>
+                        <mu2>0</mu2>
+                        <slip1>1.0</slip1>
+                        <slip2>1.0</slip2>
+                    </ode>
+                </friction>
+            </surface>
+            <origin xyz="0 0 0" rpy="0 0 0"/>
+        </collision>
         <!-- ==== FRONT LEFT CASTER WHEEL ==== -->
         <visual>
@@ -18,4 +34,20 @@
             <material name="blue"/>
         </visual>
+        <collision>
+            <geometry>
+                <mesh filename="package://robot_description/meshes/caster_wheel.stl" scale="1 1 1" />
+            </geometry>
+            <surface>
+                <friction>
+                    <ode>
+                        <mu>0</mu>
+                        <mu2>0</mu2>
+                        <slip1>1.0</slip1>
+                        <slip2>1.0</slip2>
+                    </ode>
+                </friction>
+            </surface>
+            <origin xyz="0.410295 0.24 -0.112536" rpy="0 0 0"/>
+        </collision>
         <!-- ==== FRONT RIGHT CASTER WHEEL ==== -->
         <visual>
@@ -26,4 +58,20 @@
             <material name="blue"/>
         </visual>
+        <collision>
+            <geometry>
+                <mesh filename="package://robot_description/meshes/caster_wheel.stl"  scale="1 1 1" />
+            </geometry>
+            <surface>
+                <friction>
+                    <ode>
+                        <mu>0</mu>
+                        <mu2>0</mu2>
+                        <slip1>1.0</slip1>
+                        <slip2>1.0</slip2>
+                    </ode>
+                </friction>
+            </surface>
+            <origin xyz="0.410295 -0.24 -0.112536" rpy="0 0 0"/>
+        </collision>
         <!-- ==== BACK LEFT CASTER WHEEL ==== -->
         <visual>
@@ -34,4 +82,20 @@
             <material name="blue"/>
         </visual>
+        <collision>
+            <geometry>
+                <mesh filename="package://robot_description/meshes/caster_wheel.stl"  scale="1 1 1" />
+            </geometry>
+            <surface>
+                <friction>
+                    <ode>
+                        <mu>0</mu>
+                        <mu2>0</mu2>
+                        <slip1>1.0</slip1>
+                        <slip2>1.0</slip2>
+                    </ode>
+                </friction>
+            </surface>
+            <origin xyz="-0.410295 0.24 -0.112536" rpy="0 0 0"/>
+        </collision>
         <!-- ==== BACK RIGHT CASTER WHEEL ==== -->
         <visual>
@@ -42,4 +106,20 @@
             <material name="blue"/>
         </visual>
+        <collision>
+            <geometry>
+                <mesh filename="package://robot_description/meshes/caster_wheel.stl"  scale="1 1 1" />
+            </geometry>
+            <surface>
+                <friction>
+                    <ode>
+                        <mu>0</mu>
+                        <mu2>0</mu2>
+                        <slip1>1.0</slip1>
+                        <slip2>1.0</slip2>
+                    </ode>
+                </friction>
+            </surface>
+            <origin xyz="-0.410295 -0.24 -0.112536" rpy="0 0 0"/>
+        </collision>
     </link>
 </robot>

File: robot_description/urdf/camera.xacro (robot description, xacro)
@@ -10,4 +10,10 @@
             <material name="blue"/>
         </visual>
+        <collision>
+            <geometry>
+                <mesh filename="package://robot_description/meshes/camera.stl" scale="1 1 1"  />
+            </geometry>
+            <origin xyz="0 0 0" rpy="0 0 0"/>
+        </collision>
     </link>
     <joint name="base_to_camera" type="fixed">

File: robot_description/urdf/imu.xacro (robot description, xacro)
@@ -10,4 +10,10 @@
             <material name="blue"/>
         </visual>
+        <collision>
+            <geometry>
+                <mesh filename="package://robot_description/meshes/imu.stl" scale="1 1 1"  />
+            </geometry>
+            <origin xyz="0 0 0" rpy="0 0 1.57075"/>
+        </collision>
     </link>
     <joint name="base_to_imu" type="fixed">

File: robot_description/urdf/lasers.xacro (robot description, xacro)
@@ -8,6 +8,12 @@
             </geometry>
             <origin xyz="0 0 -0.04" rpy="0 0 -0.785375"/>
-        <material name="blue"/>
+            <material name="blue"/>
         </visual>
+        <collision>
+            <geometry>
+                <mesh filename="package://robot_description/meshes/laser.stl" scale="1 1 1" />
+            </geometry>
+            <origin xyz="0 0 -0.04" rpy="0 0 -0.785375"/>
+        </collision>
     </link>
     <joint name="base_to_front_laser" type="fixed">
@@ -25,4 +31,10 @@
           <material name="blue"/>
         </visual>
+        <collision>
+            <geometry>
+                <mesh filename="package://robot_description/meshes/laser.stl" scale="1 1 1" />
+            </geometry>
+            <origin xyz="0 0 -0.04" rpy="0 0 2.355"/>
+        </collision>
     </link>
     <joint name="base_to_back_laser" type="fixed">

File: robot_description/urdf/wheels.xacro (robot description, xacro)
@@ -10,4 +10,10 @@
             <material name="blue"/>
         </visual>
+        <collision>
+            <geometry>
+                <mesh filename="package://robot_description/meshes/wheel.stl" scale="1 1 1" />
+            </geometry>
+            <origin xyz="0 0 0" rpy="0 0 0"/>
+        </collision>
     </link>
     <joint name="base_to_right_wheel" type="fixed">
@@ -25,4 +31,10 @@
             <material name="blue"/>
         </visual>
+        <collision>
+            <geometry>
+                <mesh filename="package://robot_description/meshes/wheel.stl" scale="1 1 1"  />
+            </geometry>
+            <origin xyz="0 0 0" rpy="0 0 0"/>
+        </collision>
     </link>
     <joint name="base_to_left_wheel" type="fixed">

Commit message: created no-adjusted inertial in robot_decription

File: robot_description/urdf/base_link.xacro (robot description, xacro)
@@ -26,4 +26,8 @@
             <origin xyz="0 0 0" rpy="0 0 0"/>
         </collision>
+        <inertial>
+            <mass value="5"/>
+            <inertia ixx="1.0" ixy="0.0" ixz="0.0" iyy="1.0" iyz="0.0" izz="1.0" />
+        </inertial>
         <!-- ==== FRONT LEFT CASTER WHEEL ==== -->
         <visual>

File: robot_description/urdf/camera.xacro (robot description, xacro)
@@ -16,4 +16,8 @@
             <origin xyz="0 0 0" rpy="0 0 0"/>
         </collision>
+        <inertial>
+            <mass value="0.5"/>
+            <inertia ixx="1.0" ixy="0.0" ixz="0.0" iyy="1.0" iyz="0.0" izz="1.0" />
+        </inertial>
     </link>
     <joint name="base_to_camera" type="fixed">

File: robot_description/urdf/imu.xacro (robot description, xacro)
@@ -16,4 +16,8 @@
             <origin xyz="0 0 0" rpy="0 0 1.57075"/>
         </collision>
+        <inertial>
+            <mass value="0.5"/>
+            <inertia ixx="1.0" ixy="0.0" ixz="0.0" iyy="1.0" iyz="0.0" izz="1.0" />
+        </inertial>
     </link>
     <joint name="base_to_imu" type="fixed">

File: robot_description/urdf/lasers.xacro (robot description, xacro)
@@ -7,5 +7,5 @@
                 <mesh filename="package://robot_description/meshes/laser.stl" scale="1 1 1" />
             </geometry>
-            <origin xyz="0 0 -0.04" rpy="0 0 -0.785375"/>
+            <origin xyz="0 0 -0.04" rpy="0 0 0"/>
             <material name="blue"/>
         </visual>
@@ -14,11 +14,15 @@
                 <mesh filename="package://robot_description/meshes/laser.stl" scale="1 1 1" />
             </geometry>
-            <origin xyz="0 0 -0.04" rpy="0 0 -0.785375"/>
+            <origin xyz="0 0 -0.04" rpy="0 0 0"/>
         </collision>
+        <inertial>
+            <mass value="1"/>
+            <inertia ixx="1.0" ixy="0.0" ixz="0.0" iyy="1.0" iyz="0.0" izz="1.0" />
+        </inertial>
     </link>
     <joint name="base_to_front_laser" type="fixed">
         <parent link="base_link"/>
         <child link="front_laser"/>
-        <origin xyz="0.463324 -0.251979 0.03" />
+        <origin xyz="0.463324 -0.251979 0.03" rpy="0 0 -0.785375"/>
     </joint>
     <!-- ==== BACK LASER ==== -->
@@ -28,5 +32,5 @@
                 <mesh filename="package://robot_description/meshes/laser.stl" scale="1 1 1" />
             </geometry>
-            <origin xyz="0 0 -0.04" rpy="0 0 2.355"/>
+            <origin xyz="0 0 -0.04" rpy="0 0 0"/>
           <material name="blue"/>
         </visual>
@@ -35,11 +39,15 @@
                 <mesh filename="package://robot_description/meshes/laser.stl" scale="1 1 1" />
             </geometry>
-            <origin xyz="0 0 -0.04" rpy="0 0 2.355"/>
+            <origin xyz="0 0 -0.04" rpy="0 0 0"/>
         </collision>
+        <inertial>
+            <mass value="1"/>
+            <inertia ixx="1.0" ixy="0.0" ixz="0.0" iyy="1.0" iyz="0.0" izz="1.0" />
+        </inertial>
     </link>
     <joint name="base_to_back_laser" type="fixed">
         <parent link="base_link"/>
         <child link="back_laser"/>
-        <origin xyz="-0.454597 0.230597 0.03" />
+        <origin xyz="-0.454597 0.230597 0.03" rpy="0 0 2.355"/>
     </joint>
 </robot>

File: robot_description/urdf/wheels.xacro (robot description, xacro)
@@ -16,4 +16,8 @@
             <origin xyz="0 0 0" rpy="0 0 0"/>
         </collision>
+        <inertial>
+            <mass value="1"/>
+            <inertia ixx="1.0" ixy="0.0" ixz="0.0" iyy="1.0" iyz="0.0" izz="1.0" />
+        </inertial>
     </link>
     <joint name="base_to_right_wheel" type="fixed">
@@ -37,4 +41,8 @@
             <origin xyz="0 0 0" rpy="0 0 0"/>
         </collision>
+        <inertial>
+            <mass value="1"/>
+            <inertia ixx="1.0" ixy="0.0" ixz="0.0" iyy="1.0" iyz="0.0" izz="1.0" />
+        </inertial>
     </link>
     <joint name="base_to_left_wheel" type="fixed">
