Commit message: create gazebo plugins and rviz file config

File: robot_description/urdf/camera.xacro (robot description, xacro)
@@ -1,18 +1,30 @@
 <?xml version="1.0"?>
 <robot name="robot" xmlns:xacro="http://www.ros.org/wiki/xacro">
+    <link name="front_realsense" />
+    <!--
+        The gazebo plugin aligns the depth data with the Z axis, with X=left and Y=up
+        ROS expects the depth data along the X axis, with Y=left and Z=up
+        This link only exists to give the gazebo plugin the correctly-oriented frame
+    -->
+    <link name="front_realsense_gazebo" />
+    <joint name="front_realsense_gazebo_joint" type="fixed">
+        <parent link="front_realsense"/>
+        <child link="front_realsense_gazebo"/>
+        <origin xyz="0.0 0 0" rpy="-1.5707963267948966 0 -1.5707963267948966"/>
+    </joint>
     <!-- ==== CAMERA ==== -->
     <link name="depth_camera">
         <visual>
             <geometry>
-                <mesh filename="package://robot_description/meshes/camera.stl" scale="1 1 1"  />
+                <mesh filename="package://realsense2_description/meshes/d435.dae" scale="1 1 1"  />
             </geometry>
-            <origin xyz="0 0 0" rpy="0 0 0"/>
+            <origin xyz="0 0 0" rpy="1.57075 0 1.57075"/>
             <material name="blue"/>
         </visual>
         <collision>
             <geometry>
-                <mesh filename="package://robot_description/meshes/camera.stl" scale="1 1 1"  />
+                <mesh filename="package://realsense2_description/meshes/d435.dae" scale="1 1 1"  />
             </geometry>
-            <origin xyz="0 0 0" rpy="0 0 0"/>
+            <origin xyz="0 0 0" rpy="1.57075 0 1.57075"/>
         </collision>
         <inertial>
@@ -26,3 +38,8 @@
         <origin xyz="0.523916 -0.012133 -0.03674" />
     </joint>
+    <joint type="fixed" name="front_realsense_joint">
+        <origin xyz="0.025 0 0" rpy="0 0 0" />
+        <parent link="depth_camera" />
+        <child link="front_realsense" />
+    </joint>
 </robot>

File: robot_description/urdf/lasers.xacro (robot description, xacro)
@@ -5,14 +5,14 @@
         <visual>
             <geometry>
-                <mesh filename="package://robot_description/meshes/laser.stl" scale="1 1 1" />
+                <mesh filename="package://robot_description/meshes/laser.stl" scale="0.8 0.8 0.8" />
             </geometry>
-            <origin xyz="0 0 -0.04" rpy="0 0 0"/>
+            <origin xyz="0 0 -0.09" rpy="0 0 0"/>
             <material name="blue"/>
         </visual>
         <collision>
             <geometry>
-                <mesh filename="package://robot_description/meshes/laser.stl" scale="1 1 1" />
+                <mesh filename="package://robot_description/meshes/laser.stl" scale="0.8 0.8 0.8" />
             </geometry>
-            <origin xyz="0 0 -0.04" rpy="0 0 0"/>
+            <origin xyz="0 0 -0.09" rpy="0 0 0"/>
         </collision>
         <inertial>
@@ -24,5 +24,5 @@
         <parent link="base_link"/>
         <child link="front_laser"/>
-        <origin xyz="0.463324 -0.251979 0.03" rpy="0 0 -0.785375"/>
+        <origin xyz="0.475348 -0.26853 0.07" rpy="0 0 -0.785375"/>
     </joint>
     <!-- ==== BACK LASER ==== -->
@@ -30,14 +30,14 @@
         <visual>
             <geometry>
-                <mesh filename="package://robot_description/meshes/laser.stl" scale="1 1 1" />
+                <mesh filename="package://robot_description/meshes/laser.stl" scale="0.8 0.8 0.8" />
             </geometry>
-            <origin xyz="0 0 -0.04" rpy="0 0 0"/>
+            <origin xyz="0 0 -0.09" rpy="0 0 0"/>
           <material name="blue"/>
         </visual>
         <collision>
             <geometry>
-                <mesh filename="package://robot_description/meshes/laser.stl" scale="1 1 1" />
+                <mesh filename="package://robot_description/meshes/laser.stl" scale="0.8 0.8 0.8" />
             </geometry>
-            <origin xyz="0 0 -0.04" rpy="0 0 0"/>
+            <origin xyz="0 0 -0.09" rpy="0 0 0"/>
         </collision>
         <inertial>
@@ -49,5 +49,5 @@
         <parent link="base_link"/>
         <child link="back_laser"/>
-        <origin xyz="-0.454597 0.230597 0.03" rpy="0 0 2.355"/>
+        <origin xyz="-0.474597 0.240597 0.07" rpy="0 0 2.355"/>
     </joint>
 </robot>

File: robot_description/urdf/robot.xacro (robot description, xacro)
@@ -4,4 +4,25 @@
         <color rgba="0 0 0.8 1"/>
     </material>
+    <gazebo reference="base_link">
+        <material>Gazebo/Yellow</material>
+    </gazebo>
+    <gazebo reference="front_laser">
+        <material>Gazebo/Green</material>
+    </gazebo>
+    <gazebo reference="back_laser">
+        <material>Gazebo/Green</material>
+    </gazebo>
+    <gazebo reference="left_wheel">
+        <material>Gazebo/Blue</material>
+    </gazebo>
+    <gazebo reference="right_wheel">
+        <material>Gazebo/Blue</material>
+    </gazebo>
+    <gazebo reference="depth_camera">
+        <material>Gazebo/Green</material>
+    </gazebo>
+    <gazebo reference="depth_camera">
+        <material>Gazebo/Green</material>
+    </gazebo>
     <pose>0 0 0 0 0 0</pose>
     <xacro:include filename="$(find robot_description)/urdf/base_link.xacro" />
@@ -10,3 +31,140 @@
     <xacro:include filename="$(find robot_description)/urdf/wheels.xacro" />
     <xacro:include filename="$(find robot_description)/urdf/imu.xacro" />
+    <!-- Gazebo Configurations-->
+    <gazebo>
+        <plugin name="gazebo_ros_control" filename="libgazebo_ros_control.so">
+            <robotNamespace>/</robotNamespace>
+        </plugin>
+    </gazebo>
+    <!-- IMU -->
+    <gazebo reference="imu">
+        <gravity>true</gravity>
+            <sensor name="imu_sensor" type="imu">
+            <always_on>true</always_on>
+            <update_rate>100</update_rate>
+            <visualize>true</visualize>
+            <topic>__default_topic__</topic>
+            <plugin filename="libgazebo_ros_imu_sensor.so" name="imu_plugin">
+                <topicName>imu</topicName>
+                <bodyName>imu</bodyName>
+                <updateRateHZ>10.0</updateRateHZ>
+                <gaussianNoise>0.0</gaussianNoise>
+                <xyzOffset>0 0 0</xyzOffset>
+                <rpyOffset>0 0 0</rpyOffset>
+                <frameName>imu</frameName>
+                <initialOrientationAsReference>false</initialOrientationAsReference>
+            </plugin>
+            <pose>0 0 0 0 0 0</pose>
+        </sensor>
+    </gazebo>
+    <!-- Front Sick Lidar -->
+    <gazebo reference="front_laser">
+        <sensor type="ray" name="front_lidar_sensor">
+        <pose>0 0 0 0 0 0</pose>
+        <visualize>true</visualize>
+        <update_rate>15</update_rate>
+        <ray>
+            <scan>
+            <horizontal>
+                <samples>810</samples>
+                <resolution>1</resolution>
+                <min_angle>2.356125</min_angle>
+                <max_angle>-2.356125</max_angle>
+            </horizontal>
+            </scan>
+            <range>
+            <min>0.10</min>
+            <max>25</max>
+            <resolution>0.01</resolution>
+            </range>
+            <noise>
+            <type>gaussian</type>
+            <mean>0.0</mean>
+            <stddev>0.01</stddev>
+            </noise>
+        </ray>
+        <plugin name="gazebo_ros_head_lidar_controller" filename="libgazebo_ros_laser.so">
+            <topicName>/front_scan</topicName>
+            <frameName>front_laser</frameName>
+        </plugin>
+        </sensor>
+    </gazebo>
+    <!-- Back Sick Lidar -->
+    <gazebo reference="back_laser">
+        <sensor type="ray" name="back_lidar_sensor">
+        <pose>0 0 0 0 0 0</pose>
+        <visualize>true</visualize>
+        <update_rate>15</update_rate>
+        <ray>
+            <scan>
+            <horizontal>
+                <samples>810</samples>
+                <resolution>1</resolution>
+                <min_angle>2.356125</min_angle>
+                <max_angle>-2.356125</max_angle>
+            </horizontal>
+            </scan>
+            <range>
+            <min>0.10</min>
+            <max>25</max>
+            <resolution>0.01</resolution>
+            </range>
+            <noise>
+            <type>gaussian</type>
+            <mean>0.0</mean>
+            <stddev>0.01</stddev>
+            </noise>
+        </ray>
+        <plugin name="gazebo_ros_head_lidar_controller" filename="libgazebo_ros_laser.so">
+            <topicName>/back_scan</topicName>
+            <frameName>back_laser</frameName>
+        </plugin>
+        </sensor>
+    </gazebo>
+    <!-- Realsense -->
+    <gazebo reference="front_realsense">
+        <turnGravityOff>false</turnGravityOff>
+        <sensor type="depth" name="front_realsense_depth">
+        <update_rate>30</update_rate>
+        <camera>
+            <!-- 75x65 degree FOV for the depth sensor -->
+            <horizontal_fov>1.5184351666666667</horizontal_fov>
+            <vertical_fov>1.0122901111111111</vertical_fov>
+            <image>
+            <width>640</width>
+            <height>480</height>
+            <format>R8G8B8</format>
+            </image>
+            <clip>
+            <!-- give the color sensor a maximum range of 50m so that the simulation renders nicely -->
+            <near>0.01</near>
+            <far>50.0</far>
+            </clip>
+        </camera>
+        <plugin name="kinect_controller" filename="libgazebo_ros_openni_kinect.so">
+            <baseline>0.2</baseline>
+            <alwaysOn>true</alwaysOn>
+            <updateRate>30</updateRate>
+            <cameraName>realsense</cameraName>
+            <imageTopicName>color/image_raw</imageTopicName>
+            <cameraInfoTopicName>color/camera_info</cameraInfoTopicName>
+            <depthImageTopicName>depth/image_rect_raw</depthImageTopicName>
+            <depthImageInfoTopicName>depth/camera_info</depthImageInfoTopicName>
+            <pointCloudTopicName>depth/color/points</pointCloudTopicName>
+            <frameName>front_realsense_gazebo</frameName>
+            <pointCloudCutoff>0.105</pointCloudCutoff>
+            <pointCloudCutoffMax>8.0</pointCloudCutoffMax>
+            <distortionK1>0.00000001</distortionK1>
+            <distortionK2>0.00000001</distortionK2>
+            <distortionK3>0.00000001</distortionK3>
+            <distortionT1>0.00000001</distortionT1>
+            <distortionT2>0.00000001</distortionT2>
+            <CxPrime>0</CxPrime>
+            <Cx>0</Cx>
+            <Cy>0</Cy>
+            <focalLength>0</focalLength>
+            <hackBaseline>0</hackBaseline>
+        </plugin>
+        </sensor>
+    </gazebo>
 </robot>

Commit message: create teleop configuration

File: robot_description/urdf/camera.xacro (robot description, xacro)
@@ -1,16 +1,4 @@
 <?xml version="1.0"?>
 <robot name="robot" xmlns:xacro="http://www.ros.org/wiki/xacro">
-    <link name="front_realsense" />
-    <!--
-        The gazebo plugin aligns the depth data with the Z axis, with X=left and Y=up
-        ROS expects the depth data along the X axis, with Y=left and Z=up
-        This link only exists to give the gazebo plugin the correctly-oriented frame
-    -->
-    <link name="front_realsense_gazebo" />
-    <joint name="front_realsense_gazebo_joint" type="fixed">
-        <parent link="front_realsense"/>
-        <child link="front_realsense_gazebo"/>
-        <origin xyz="0.0 0 0" rpy="-1.5707963267948966 0 -1.5707963267948966"/>
-    </joint>
     <!-- ==== CAMERA ==== -->
     <link name="depth_camera">
@@ -29,6 +17,6 @@
         </collision>
         <inertial>
-            <mass value="0.5"/>
-            <inertia ixx="1.0" ixy="0.0" ixz="0.0" iyy="1.0" iyz="0.0" izz="1.0" />
+            <mass value="0.01"/>
+            <inertia ixx="0.01" ixy="0.0" ixz="0.0" iyy="0.01" iyz="0.0" izz="0.01" />
         </inertial>
     </link>
@@ -38,4 +26,5 @@
         <origin xyz="0.523916 -0.012133 -0.03674" />
     </joint>
+    <link name="front_realsense" />
     <joint type="fixed" name="front_realsense_joint">
         <origin xyz="0.025 0 0" rpy="0 0 0" />
@@ -43,3 +32,14 @@
         <child link="front_realsense" />
     </joint>
+     <!--
+        The gazebo plugin aligns the depth data with the Z axis, with X=left and Y=up
+        ROS expects the depth data along the X axis, with Y=left and Z=up
+        This link only exists to give the gazebo plugin the correctly-oriented frame
+    -->
+    <link name="front_realsense_gazebo" />
+    <joint name="front_realsense_gazebo_joint" type="fixed">
+        <parent link="front_realsense"/>
+        <child link="front_realsense_gazebo"/>
+        <origin xyz="0.0 0 0" rpy="-1.5707963267948966 0 -1.5707963267948966"/>
+    </joint>
 </robot>

File: robot_description/urdf/imu.xacro (robot description, xacro)
@@ -17,6 +17,6 @@
         </collision>
         <inertial>
-            <mass value="0.5"/>
-            <inertia ixx="1.0" ixy="0.0" ixz="0.0" iyy="1.0" iyz="0.0" izz="1.0" />
+            <mass value="0.02"/>
+            <inertia ixx="0.01" ixy="0.0" ixz="0.0" iyy="0.01" iyz="0.0" izz="0.01" />
         </inertial>
     </link>

File: robot_description/urdf/lasers.xacro (robot description, xacro)
@@ -18,5 +18,5 @@
         <inertial>
             <mass value="1"/>
-            <inertia ixx="1.0" ixy="0.0" ixz="0.0" iyy="1.0" iyz="0.0" izz="1.0" />
+            <inertia ixx="0.01" ixy="0.0" ixz="0.0" iyy="0.01" iyz="0.0" izz="0.01" />
         </inertial>
     </link>
@@ -43,5 +43,5 @@
         <inertial>
             <mass value="1"/>
-            <inertia ixx="1.0" ixy="0.0" ixz="0.0" iyy="1.0" iyz="0.0" izz="1.0" />
+            <inertia ixx="0.01" ixy="0.0" ixz="0.0" iyy="0.01" iyz="0.0" izz="0.01" />
         </inertial>
     </link>

File: robot_description/urdf/robot.xacro (robot description, xacro)
@@ -4,167 +4,14 @@
         <color rgba="0 0 0.8 1"/>
     </material>
-    <gazebo reference="base_link">
-        <material>Gazebo/Yellow</material>
-    </gazebo>
-    <gazebo reference="front_laser">
-        <material>Gazebo/Green</material>
-    </gazebo>
-    <gazebo reference="back_laser">
-        <material>Gazebo/Green</material>
-    </gazebo>
-    <gazebo reference="left_wheel">
-        <material>Gazebo/Blue</material>
-    </gazebo>
-    <gazebo reference="right_wheel">
-        <material>Gazebo/Blue</material>
-    </gazebo>
-    <gazebo reference="depth_camera">
-        <material>Gazebo/Green</material>
-    </gazebo>
-    <gazebo reference="depth_camera">
-        <material>Gazebo/Green</material>
-    </gazebo>
     <pose>0 0 0 0 0 0</pose>
-    <xacro:include filename="$(find robot_description)/urdf/base_link.xacro" />
+    <xacro:include filename="$(find robot_description)/gazebo/ros_control.gazebo" />
+    <xacro:include filename="$(find robot_description)/gazebo/diff_driver.gazebo" />
+    <xacro:include filename="$(find robot_description)/gazebo/imu.gazebo" />
+    <xacro:include filename="$(find robot_description)/gazebo/lasers.gazebo" />
+    <xacro:include filename="$(find robot_description)/gazebo/camera.gazebo" />
+    <xacro:include filename="$(find robot_description)/urdf/base.xacro" />
     <xacro:include filename="$(find robot_description)/urdf/camera.xacro" />
     <xacro:include filename="$(find robot_description)/urdf/lasers.xacro" />
     <xacro:include filename="$(find robot_description)/urdf/wheels.xacro" />
     <xacro:include filename="$(find robot_description)/urdf/imu.xacro" />
-    <!-- Gazebo Configurations-->
-    <gazebo>
-        <plugin name="gazebo_ros_control" filename="libgazebo_ros_control.so">
-            <robotNamespace>/</robotNamespace>
-        </plugin>
-    </gazebo>
-    <!-- IMU -->
-    <gazebo reference="imu">
-        <gravity>true</gravity>
-            <sensor name="imu_sensor" type="imu">
-            <always_on>true</always_on>
-            <update_rate>100</update_rate>
-            <visualize>true</visualize>
-            <topic>__default_topic__</topic>
-            <plugin filename="libgazebo_ros_imu_sensor.so" name="imu_plugin">
-                <topicName>imu</topicName>
-                <bodyName>imu</bodyName>
-                <updateRateHZ>10.0</updateRateHZ>
-                <gaussianNoise>0.0</gaussianNoise>
-                <xyzOffset>0 0 0</xyzOffset>
-                <rpyOffset>0 0 0</rpyOffset>
-                <frameName>imu</frameName>
-                <initialOrientationAsReference>false</initialOrientationAsReference>
-            </plugin>
-            <pose>0 0 0 0 0 0</pose>
-        </sensor>
-    </gazebo>
-    <!-- Front Sick Lidar -->
-    <gazebo reference="front_laser">
-        <sensor type="ray" name="front_lidar_sensor">
-        <pose>0 0 0 0 0 0</pose>
-        <visualize>true</visualize>
-        <update_rate>15</update_rate>
-        <ray>
-            <scan>
-            <horizontal>
-                <samples>810</samples>
-                <resolution>1</resolution>
-                <min_angle>2.356125</min_angle>
-                <max_angle>-2.356125</max_angle>
-            </horizontal>
-            </scan>
-            <range>
-            <min>0.10</min>
-            <max>25</max>
-            <resolution>0.01</resolution>
-            </range>
-            <noise>
-            <type>gaussian</type>
-            <mean>0.0</mean>
-            <stddev>0.01</stddev>
-            </noise>
-        </ray>
-        <plugin name="gazebo_ros_head_lidar_controller" filename="libgazebo_ros_laser.so">
-            <topicName>/front_scan</topicName>
-            <frameName>front_laser</frameName>
-        </plugin>
-        </sensor>
-    </gazebo>
-    <!-- Back Sick Lidar -->
-    <gazebo reference="back_laser">
-        <sensor type="ray" name="back_lidar_sensor">
-        <pose>0 0 0 0 0 0</pose>
-        <visualize>true</visualize>
-        <update_rate>15</update_rate>
-        <ray>
-            <scan>
-            <horizontal>
-                <samples>810</samples>
-                <resolution>1</resolution>
-                <min_angle>2.356125</min_angle>
-                <max_angle>-2.356125</max_angle>
-            </horizontal>
-            </scan>
-            <range>
-            <min>0.10</min>
-            <max>25</max>
-            <resolution>0.01</resolution>
-            </range>
-            <noise>
-            <type>gaussian</type>
-            <mean>0.0</mean>
-            <stddev>0.01</stddev>
-            </noise>
-        </ray>
-        <plugin name="gazebo_ros_head_lidar_controller" filename="libgazebo_ros_laser.so">
-            <topicName>/back_scan</topicName>
-            <frameName>back_laser</frameName>
-        </plugin>
-        </sensor>
-    </gazebo>
-    <!-- Realsense -->
-    <gazebo reference="front_realsense">
-        <turnGravityOff>false</turnGravityOff>
-        <sensor type="depth" name="front_realsense_depth">
-        <update_rate>30</update_rate>
-        <camera>
-            <!-- 75x65 degree FOV for the depth sensor -->
-            <horizontal_fov>1.5184351666666667</horizontal_fov>
-            <vertical_fov>1.0122901111111111</vertical_fov>
-            <image>
-            <width>640</width>
-            <height>480</height>
-            <format>R8G8B8</format>
-            </image>
-            <clip>
-            <!-- give the color sensor a maximum range of 50m so that the simulation renders nicely -->
-            <near>0.01</near>
-            <far>50.0</far>
-            </clip>
-        </camera>
-        <plugin name="kinect_controller" filename="libgazebo_ros_openni_kinect.so">
-            <baseline>0.2</baseline>
-            <alwaysOn>true</alwaysOn>
-            <updateRate>30</updateRate>
-            <cameraName>realsense</cameraName>
-            <imageTopicName>color/image_raw</imageTopicName>
-            <cameraInfoTopicName>color/camera_info</cameraInfoTopicName>
-            <depthImageTopicName>depth/image_rect_raw</depthImageTopicName>
-            <depthImageInfoTopicName>depth/camera_info</depthImageInfoTopicName>
-            <pointCloudTopicName>depth/color/points</pointCloudTopicName>
-            <frameName>front_realsense_gazebo</frameName>
-            <pointCloudCutoff>0.105</pointCloudCutoff>
-            <pointCloudCutoffMax>8.0</pointCloudCutoffMax>
-            <distortionK1>0.00000001</distortionK1>
-            <distortionK2>0.00000001</distortionK2>
-            <distortionK3>0.00000001</distortionK3>
-            <distortionT1>0.00000001</distortionT1>
-            <distortionT2>0.00000001</distortionT2>
-            <CxPrime>0</CxPrime>
-            <Cx>0</Cx>
-            <Cy>0</Cy>
-            <focalLength>0</focalLength>
-            <hackBaseline>0</hackBaseline>
-        </plugin>
-        </sensor>
-    </gazebo>
 </robot>

File: robot_description/urdf/wheels.xacro (robot description, xacro)
@@ -18,11 +18,14 @@
         <inertial>
             <mass value="1"/>
-            <inertia ixx="1.0" ixy="0.0" ixz="0.0" iyy="1.0" iyz="0.0" izz="1.0" />
+            <inertia ixx="0.01" ixy="0.0" ixz="0.0" iyy="0.01" iyz="0.0" izz="0.01" />
         </inertial>
     </link>
-    <joint name="base_to_right_wheel" type="fixed">
+    <joint name="base_to_right_wheel" type="continuous">
         <parent link="base_link"/>
         <child link="right_wheel"/>
-        <origin xyz="-0.007 -0.24 -0.18" />
+        <origin xyz="-0.007 -0.24 -0.1801" />
+        <axis rpy="0 0 0" xyz="0 1 0"/>
+        <limit effort="10000" velocity="1000"/>
+        <joint_properties damping="1.0" friction="1.0"/>
     </joint>
     <!-- ==== LEFT WHEEL ==== -->
@@ -43,11 +46,14 @@
         <inertial>
             <mass value="1"/>
-            <inertia ixx="1.0" ixy="0.0" ixz="0.0" iyy="1.0" iyz="0.0" izz="1.0" />
+            <inertia ixx="0.01" ixy="0.0" ixz="0.0" iyy="0.01" iyz="0.0" izz="0.01" />
         </inertial>
     </link>
-    <joint name="base_to_left_wheel" type="fixed">
+    <joint name="base_to_left_wheel" type="continuous">
         <parent link="base_link"/>
         <child link="left_wheel"/>
-        <origin xyz="-0.007 0.24 -0.18" />
+        <origin xyz="-0.007 0.24 -0.1801" />
+        <axis rpy="0 0 0" xyz="0 1 0"/>
+        <limit effort="10000" velocity="1000"/>
+        <joint_properties damping="1.0" friction="1.0"/>
     </joint>
 </robot>
